File: HW/OLED_1_3INCH_I2C.brd (EAGLE design)
At the start: 35.5 x 33.5 mm, 31 parts, among them IC1 ME6211C33M5G

Commit message: new
Parts:
- D1: device diode:SOD323-R -> LasKKit-Discrete:SOD323-R
Routing:
- net GND: track 1.22 -> 0.00 mm
- net +3V3: track 100.4 -> 99.8 mm
Changed lines of the file:
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@@
 <drawing>
 <settings>
-<setting alwaysvectorfont="yes"/>
+<setting alwaysvectorfont="no"/>
 <setting verticaltext="up"/>
 </settings>
@@
 <layer number="156" name="tAssmbl" color="7" fill="1" visible="no" active="yes"/>
 <layer number="157" name="bAssmbl" color="7" fill="1" visible="no" active="yes"/>
+<layer number="158" name="FaceMMeas" color="7" fill="1" visible="no" active="no"/>
+<layer number="159" name="Geh-Bear2" color="7" fill="1" visible="no" active="no"/>
+<layer number="160" name="Topologie" color="7" fill="1" visible="no" active="no"/>
+<layer number="161" name="tomplace2" color="7" fill="1" visible="no" active="no"/>
 <layer number="166" name="AntennaArea" color="7" fill="1" visible="no" active="yes"/>
 <layer number="168" name="4mmHeightArea" color="7" fill="1" visible="no" active="yes"/>
@@
 <layer number="250" name="Descript" color="7" fill="1" visible="no" active="yes"/>
 <layer number="251" name="SMDround" color="7" fill="1" visible="no" active="yes"/>
+<layer number="252" name="BR-BS" color="7" fill="1" visible="no" active="no"/>
+<layer number="253" name="Extra" color="7" fill="1" visible="no" active="no"/>
 <layer number="254" name="cooling" color="7" fill="1" visible="no" active="yes"/>
 <layer number="255" name="routoute" color="7" fill="1" visible="no" active="yes"/>
 </layers>
 <board>
+<fusionsync huburn="a.cGVyc29uYWw6dWUyODMwMzEw" projecturn="a.cGVyc29uYWw6dWUyODMwMzEwIzIwMjAxMjA0MzU5NTU4Nzc2" f3durn="urn:adsk.wipprod:dm.lineage:JgbjurpjT7CtaIdP9RWt-Q" pcbguid="" lastpulledtime="" lastsyncedchangeguid="" latestrevisionid="8ab12d7c-35e5-424c-8579-8515671fbc90" lastsyncedrevisionid="8ab12d7c-35e5-424c-8579-8515671fbc90" lastboardhashguid="eecc9839-aaa1-8b0d-51ec-a875e29f6833" lastpushedtime="2023-01-27T11:16:59Z" linktopcb3d="true"/>
 <plain>
 <wire x1="2.5" y1="0" x2="10.5" y2="0" width="0" layer="20"/>
@@
 <attribute name="VALUE" x="14.1478" y="30.861" size="1.27" layer="28" rot="MR180"/>
 </element>
-<element name="D1" library="diode" library_urn="urn:adsk.eagle:library:210" package="SOD323-R" package3d_urn="urn:adsk.eagle:package:43437/1" value="1N4148" x="14.6812" y="19.6596" smashed="yes" rot="MR270">
+<element name="D1" library="LasKKit-Discrete" library_urn="urn:adsk.eagle:library:27330413" package="SOD323-R" package3d_urn="urn:adsk.eagle:package:37888618/2" value="1N4148" x="14.6812" y="19.6596" smashed="yes" rot="MR270">
+<attribute name="LCSC_PART" value="" x="14.6812" y="19.6596" size="1.778" layer="28" rot="MR270" display="off"/>
 <attribute name="NAME" x="14.6988" y="21.7838" size="0.8128" layer="26" font="vector" ratio="15" rot="MR180" align="center"/>
-<attribute name="POPULARITY" value="4" x="43.8912" y="-7.0104" size="1.778" layer="28" rot="MR270" display="off"/>
 <attribute name="VALUE" x="16.9812" y="20.7596" size="1.27" layer="28" rot="MR270"/>
 </element>
-<element name="DISPLAY1" library="LasKKit-Displays" library_urn="urn:adsk.eagle:library:27617220" package="GME12864_1_3INCH" package3d_urn="urn:adsk.eagle:package:35641174/4" value="OLED_1_3INCH" x="17.75" y="16.75" smashed="yes">
+<element name="DISPLAY1" library="LasKKit-Displays" library_urn="urn:adsk.eagle:library:27617220" package="GME12864_1_3INCH" package3d_urn="urn:adsk.eagle:package:35641174/8" value="OLED_1_3INCH" x="17.75" y="16.75" smashed="yes">
 <attribute name="NAME" x="17.75" y="16.5" size="0.8128" layer="25" font="vector" ratio="15" align="center"/>
 <attribute name="VALUE" x="17.75" y="15.25" size="0.8128" layer="27" font="vector" ratio="15" align="center"/>
 </element>
-<element name="H1" library="LasKKit-Holes" library_urn="urn:adsk.eagle:library:22988445" package="2,5-PAD" package3d_urn="urn:adsk.eagle:package:32492771/2" value="MOUNT-PAD-ROUND2.5" x="33" y="2.5" smashed="yes"/>
-<element name="H2" library="LasKKit-Holes" library_urn="urn:adsk.eagle:library:22988445" package="2,5-PAD" package3d_urn="urn:adsk.eagle:package:32492771/2" value="MOUNT-PAD-ROUND2.5" x="2.5" y="2.5" smashed="yes"/>
-<element name="H3" library="LasKKit-Holes" library_urn="urn:adsk.eagle:library:22988445" package="2,5-PAD" package3d_urn="urn:adsk.eagle:package:32492771/2" value="MOUNT-PAD-ROUND2.5" x="33" y="31" smashed="yes"/>
-<element name="H4" library="LasKKit-Holes" library_urn="urn:adsk.eagle:library:22988445" package="2,5-PAD" package3d_urn="urn:adsk.eagle:package:32492771/2" value="MOUNT-PAD-ROUND2.5" x="2.5" y="31" smashed="yes"/>
-<element name="J1" library="LasKKit-Connectors" library_urn="urn:adsk.eagle:library:21740355" package="1X04_1MM_RA" package3d_urn="urn:adsk.eagle:package:33537550/10" value="" x="28.0482" y="21.9456" smashed="yes" rot="MR90">
+<element name="H1" library="LasKKit-Holes" library_urn="urn:adsk.eagle:library:22988445" package="2,5-PAD" package3d_urn="urn:adsk.eagle:package:32492771/3" value="MOUNT-PAD-ROUND2.5" x="33" y="2.5" smashed="yes"/>
+<element name="H2" library="LasKKit-Holes" library_urn="urn:adsk.eagle:library:22988445" package="2,5-PAD" package3d_urn="urn:adsk.eagle:package:32492771/3" value="MOUNT-PAD-ROUND2.5" x="2.5" y="2.5" smashed="yes"/>
+<element name="H3" library="LasKKit-Holes" library_urn="urn:adsk.eagle:library:22988445" package="2,5-PAD" package3d_urn="urn:adsk.eagle:package:32492771/3" value="MOUNT-PAD-ROUND2.5" x="33" y="31" smashed="yes"/>
+<element name="H4" library="LasKKit-Holes" library_urn="urn:adsk.eagle:library:22988445" package="2,5-PAD" package3d_urn="urn:adsk.eagle:package:32492771/3" value="MOUNT-PAD-ROUND2.5" x="2.5" y="31" smashed="yes"/>
+<element name="J1" library="LasKKit-Connectors" library_urn="urn:adsk.eagle:library:21740355" package="1X04_1MM_RA" package3d_urn="urn:adsk.eagle:package:33537550/14" value="" x="28.0482" y="21.9456" smashed="yes" rot="MR90">
 <attribute name="LCSC_PART" value="C145956" x="0.1082" y="54.9656" size="1.778" layer="28" rot="MR90" display="off"/>
 <attribute name="NAME" x="29.7444" y="21.7932" size="0.8128" layer="26" font="vector" ratio="15" rot="MR270" align="center"/>
 <attribute name="VALUE" x="29.7952" y="23.5966" size="0.6096" layer="28" font="vector" ratio="20" rot="MR270"/>
 </element>
-<element name="J2" library="LasKKit-Connectors" library_urn="urn:adsk.eagle:library:21740355" package="1X04_1MM_RA" package3d_urn="urn:adsk.eagle:package:33537550/10" value="" x="7.4356" y="21.9456" smashed="yes" rot="MR270">
+<element name="J2" library="LasKKit-Connectors" library_urn="urn:adsk.eagle:library:21740355" package="1X04_1MM_RA" package3d_urn="urn:adsk.eagle:package:33537550/14" value="" x="7.4356" y="21.9456" smashed="yes" rot="MR270">
 <attribute name="LCSC_PART" value="C145956" x="35.3756" y="-18.6944" size="1.778" layer="28" rot="MR270" display="off"/>
 <attribute name="NAME" x="5.714" y="21.9456" size="0.8128" layer="26" font="vector" ratio="15" rot="MR90" align="center"/>
@@
 </polygon>
 <contactref element="IC1" pad="2"/>
-<wire x1="12.3998" y1="26.1874" x2="11.176" y2="26.1874" width="0.4064" layer="16"/>
 <contactref element="I2C_ADDR" pad="3"/>
 </signal>
@@
 <wire x1="17.8874" y1="20.7596" x2="14.6812" y2="20.7596" width="0.254" layer="16"/>
 <wire x1="13.6398" y1="15.2232" x2="13.6398" y2="20.7518" width="0.4064" layer="16"/>
-<wire x1="8.9906" y1="21.4456" x2="8.4328" y2="21.4456" width="0.4064" layer="16"/>
 <wire x1="8.9906" y1="21.4456" x2="12.9714" y2="21.4456" width="0.4064" layer="16"/>
 <wire x1="12.9714" y1="21.4456" x2="13.6652" y2="20.7518" width="0.4064" layer="16"/>
@@
 <mfgpreviewcolor name="substratecolor" color="0xFF786E46"/>
 </mfgpreviewcolors>
+<errors>
+</errors>
 </board>
 </drawing>
@@
 </note>
 <note version="8.3" severity="warning">
+Since Version 8.3, EAGLE supports Fusion synchronisation.
+This feature will not be available in this version and saving
+the document will break the link to the Fusion PCB feature.
+</note>
+<note version="8.3" severity="warning">

Commit message: new version
Parts:
- added I2C_PULLUPS: JUMPER-SMT_2_NC_TRACE_SILK, LaskaKit-Jumpers:SMT-JUMPER_2_NC_TRACE_SILK
- U$4: value LASKKIT_LOGO_NAME -> (none)
- moved U$4 2.01 mm to (20.7, 28.0)
- turned R5 to 180 degrees
Connections:
- new net N$12: I2C_PULLUPS.1, R5.1, R6.1
- net +3V3: now also I2C_PULLUPS.2; no longer R5.2, R6.1
- net SCL: now also R5.2; no longer R5.1
Routing:
- net N$12: track 0.00 -> 18.3 mm, vias 0 -> 2
- net +3V3: track 99.8 -> 102.1 mm
- net SCL: track 43.3 -> 44.0 mm
- net GND: track 0.00 -> 0.61 mm
Other:
- board text added: "v1.2"
- board text removed: "v1.1"
