File: HW/OLED_1_3INCH_I2C.sch (EAGLE design)
At the start: 28 parts, among them IC1 ME6211C33M5G

Commit message: new
Parts:
- D1: device diode:DIODE-SOD323-R -> LasKKit-Discrete:DIODE-SOD323-R
- J1, J2: device LasKKit-Connectors:USUP_CONNECTORHOR -> LasKKit-Connectors:USUP_CONNECTOR_HOR
Changed lines of the file:
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@@
 <layer number="156" name="tAssmbl" color="7" fill="1" visible="yes" active="yes"/>
 <layer number="157" name="bAssmbl" color="7" fill="1" visible="yes" active="yes"/>
+<layer number="158" name="FaceMMeas" color="7" fill="1" visible="no" active="no"/>
+<layer number="159" name="Geh-Bear2" color="7" fill="1" visible="no" active="no"/>
+<layer number="160" name="Topologie" color="7" fill="1" visible="no" active="no"/>
+<layer number="161" name="tomplace2" color="7" fill="1" visible="no" active="no"/>
 <layer number="166" name="AntennaArea" color="7" fill="1" visible="yes" active="yes"/>
 <layer number="168" name="4mmHeightArea" color="7" fill="1" visible="yes" active="yes"/>
@@
 <layer number="250" name="Descript" color="7" fill="1" visible="yes" active="yes"/>
 <layer number="251" name="SMDround" color="7" fill="1" visible="yes" active="yes"/>
+<layer number="252" name="BR-BS" color="7" fill="1" visible="no" active="no"/>
+<layer number="253" name="Extra" color="7" fill="1" visible="no" active="no"/>
 <layer number="254" name="cooling" color="7" fill="1" visible="yes" active="yes"/>
 <layer number="255" name="routoute" color="7" fill="1" visible="yes" active="yes"/>
@@
 </classes>
 <parts>
-<part name="DISPLAY1" library="LasKKit-Displays" library_urn="urn:adsk.eagle:library:27617220" deviceset="OLED_1_3INCH" device="" package3d_urn="urn:adsk.eagle:package:35641174/4"/>
+<part name="DISPLAY1" library="LasKKit-Displays" library_urn="urn:adsk.eagle:library:27617220" deviceset="OLED_1_3INCH" device="" package3d_urn="urn:adsk.eagle:package:35641174/8"/>
 <part name="GND1" library="supply1" library_urn="urn:adsk.eagle:library:371" deviceset="GND" device=""/>
 <part name="C1" library="rcl" library_urn="urn:adsk.eagle:library:334" deviceset="C-EU" device="C0603" package3d_urn="urn:adsk.eagle:package:23616/2" value="1uF"/>
@@
 <part name="R4" library="rcl" library_urn="urn:adsk.eagle:library:334" deviceset="R-EU_" device="R0603" package3d_urn="urn:adsk.eagle:package:23555/3" value="10k"/>
 <part name="+3V2" library="supply1" library_urn="urn:adsk.eagle:library:371" deviceset="+3V3" device=""/>
-<part name="D1" library="diode" library_urn="urn:adsk.eagle:library:210" deviceset="DIODE-" device="SOD323-R" package3d_urn="urn:adsk.eagle:package:43437/1" value="1N4148"/>
+<part name="D1" library="LasKKit-Discrete" library_urn="urn:adsk.eagle:library:27330413" deviceset="DIODE-" device="SOD323-R" package3d_urn="urn:adsk.eagle:package:37888618/2" value="1N4148"/>
 <part name="R5" library="rcl" library_urn="urn:adsk.eagle:library:334" deviceset="R-EU_" device="R0603" package3d_urn="urn:adsk.eagle:package:23555/3" value="10k"/>
 <part name="R6" library="rcl" library_urn="urn:adsk.eagle:library:334" deviceset="R-EU_" device="R0603" package3d_urn="urn:adsk.eagle:package:23555/3" value="10k"/>
@@
 <part name="C10" library="rcl" library_urn="urn:adsk.eagle:library:334" deviceset="C-EU" device="C0603" package3d_urn="urn:adsk.eagle:package:23616/2" value="22uF"/>
 <part name="JP1" library="LasKKit-Connectors" library_urn="urn:adsk.eagle:library:21740355" deviceset="PINHD-1X4" device="" package3d_urn="urn:adsk.eagle:package:21740534/1"/>
-<part name="J1" library="LasKKit-Connectors" library_urn="urn:adsk.eagle:library:21740355" deviceset="USUP_CONNECTOR" device="HOR" package3d_urn="urn:adsk.eagle:package:33537550/10"/>
-<part name="J2" library="LasKKit-Connectors" library_urn="urn:adsk.eagle:library:21740355" deviceset="USUP_CONNECTOR" device="HOR" package3d_urn="urn:adsk.eagle:package:33537550/10"/>
+<part name="J1" library="LasKKit-Connectors" library_urn="urn:adsk.eagle:library:21740355" deviceset="USUP_CONNECTOR" device="_HOR" package3d_urn="urn:adsk.eagle:package:33537550/14"/>
+<part name="J2" library="LasKKit-Connectors" library_urn="urn:adsk.eagle:library:21740355" deviceset="USUP_CONNECTOR" device="_HOR" package3d_urn="urn:adsk.eagle:package:33537550/14"/>
 <part name="P+1" library="supply1" library_urn="urn:adsk.eagle:library:371" deviceset="VCC" device=""/>
 <part name="+3V4" library="supply1" library_urn="urn:adsk.eagle:library:371" deviceset="+3V3" device=""/>
 <part name="GND3" library="supply1" library_urn="urn:adsk.eagle:library:371" deviceset="GND" device=""/>
-<part name="H1" library="LasKKit-Holes" library_urn="urn:adsk.eagle:library:22988445" deviceset="MOUNT-PAD-ROUND" device="2.5" package3d_urn="urn:adsk.eagle:package:32492771/2"/>
-<part name="H2" library="LasKKit-Holes" library_urn="urn:adsk.eagle:library:22988445" deviceset="MOUNT-PAD-ROUND" device="2.5" package3d_urn="urn:adsk.eagle:package:32492771/2"/>
-<part name="H3" library="LasKKit-Holes" library_urn="urn:adsk.eagle:library:22988445" deviceset="MOUNT-PAD-ROUND" device="2.5" package3d_urn="urn:adsk.eagle:package:32492771/2"/>
-<part name="H4" library="LasKKit-Holes" library_urn="urn:adsk.eagle:library:22988445" deviceset="MOUNT-PAD-ROUND" device="2.5" package3d_urn="urn:adsk.eagle:package:32492771/2"/>
+<part name="H1" library="LasKKit-Holes" library_urn="urn:adsk.eagle:library:22988445" deviceset="MOUNT-PAD-ROUND" device="2.5" package3d_urn="urn:adsk.eagle:package:32492771/3"/>
+<part name="H2" library="LasKKit-Holes" library_urn="urn:adsk.eagle:library:22988445" deviceset="MOUNT-PAD-ROUND" device="2.5" package3d_urn="urn:adsk.eagle:package:32492771/3"/>
+<part name="H3" library="LasKKit-Holes" library_urn="urn:adsk.eagle:library:22988445" deviceset="MOUNT-PAD-ROUND" device="2.5" package3d_urn="urn:adsk.eagle:package:32492771/3"/>
+<part name="H4" library="LasKKit-Holes" library_urn="urn:adsk.eagle:library:22988445" deviceset="MOUNT-PAD-ROUND" device="2.5" package3d_urn="urn:adsk.eagle:package:32492771/3"/>
 <part name="GND4" library="supply1" library_urn="urn:adsk.eagle:library:371" deviceset="GND" device=""/>
 <part name="FRAME1" library="LasKKit-Aesthetics" library_urn="urn:adsk.eagle:library:19472811" deviceset="FRAME-A4L" device="">
@@
 <attribute name="VALUE" x="191.77" y="86.36" size="1.778" layer="96" rot="R90"/>
 </instance>
-<instance part="J1" gate="J1" x="205.74" y="69.215" smashed="yes" rot="MR0">
+<instance part="J1" gate="A" x="205.74" y="69.215" smashed="yes" rot="MR0">
 <attribute name="VALUE" x="210.82" y="63.881" size="1.778" layer="96" font="vector" rot="MR0" align="top-left"/>
 <attribute name="NAME" x="210.82" y="77.089" size="1.778" layer="95" rot="MR0"/>
 </instance>
-<instance part="J2" gate="J1" x="158.75" y="69.215" smashed="yes">
+<instance part="J2" gate="A" x="158.75" y="69.215" smashed="yes">
 <attribute name="VALUE" x="153.67" y="63.881" size="1.778" layer="96" font="vector" align="top-left"/>
 <attribute name="NAME" x="153.67" y="77.089" size="1.778" layer="95"/>
@@
 </segment>
 <segment>
-<pinref part="J2" gate="J1" pin="GND"/>
-<pinref part="J1" gate="J1" pin="GND"/>
+<pinref part="J2" gate="A" pin="GND"/>
+<pinref part="J1" gate="A" pin="GND"/>
 <wire x1="166.37" y1="66.675" x2="169.545" y2="66.675" width="0.1524" layer="91"/>
 <pinref part="JP1" gate="A" pin="2"/>
@@
 </segment>
 <segment>
-<pinref part="J2" gate="J1" pin="VCC"/>
-<pinref part="J1" gate="J1" pin="VCC"/>
+<pinref part="J2" gate="A" pin="VCC"/>
+<pinref part="J1" gate="A" pin="VCC"/>
 <wire x1="166.37" y1="69.215" x2="169.545" y2="69.215" width="0.1524" layer="91"/>
 <pinref part="+3V4" gate="G$1" pin="+3V3"/>
@@
 </segment>
 <segment>
-<pinref part="J2" gate="J1" pin="SDA"/>
-<pinref part="J1" gate="J1" pin="SDA"/>
+<pinref part="J2" gate="A" pin="SDA"/>
+<pinref part="J1" gate="A" pin="SDA"/>
 <wire x1="166.37" y1="71.755" x2="186.69" y2="71.755" width="0.1524" layer="91"/>
 <pinref part="JP1" gate="A" pin="4"/>
@@
 </segment>
 <segment>
-<pinref part="J2" gate="J1" pin="SCL"/>
-<pinref part="J1" gate="J1" pin="SCL"/>
+<pinref part="J2" gate="A" pin="SCL"/>
+<pinref part="J1" gate="A" pin="SCL"/>
 <wire x1="166.37" y1="74.295" x2="184.15" y2="74.295" width="0.1524" layer="91"/>
 <pinref part="JP1" gate="A" pin="3"/>

Commit message: new version
Parts:
- removed U$4: LASKKIT_LOGO_NAME, LasKKit-Aesthetics:LASKKIT_LOGO_NAME
- added I2C_PULLUPS: JUMPER-SMT_2_NC_TRACE_SILK, LaskaKit-Jumpers:JUMPER-SMT_2_NC_TRACE_SILK
Connections:
- new net N$12: I2C_PULLUPS.1, R5.1, R6.1
- net +3V3: now also I2C_PULLUPS.2; no longer R5.2, R6.1
- net SCL: now also R5.2; no longer R5.1
Other:
- moved on the sheet: R5, R6
